File: design/kicad/ata-ide.kicad_pcb (KiCad board)
At the start: 2 copper layers, 81.9 x 113 mm, 32 parts, among them J1 Conn_02x32_Odd_Even, J2 Conn_02x20_Odd_Even, Q1 2N2907, U1 16V8, U2 ATF750, U3 74HCT241, U4 74HCT245, U5 74HCT245

Commit message: Update for version 1.1.
Parts:
- removed REF***: OSHW-Logo2_7.3x6mm_SilkScreen, Symbols:OSHW-Logo2_7.3x6mm_SilkScreen
- removed REF***: WEEE-Logo_4.2x6mm_SilkScreen, Symbols:WEEE-Logo_4.2x6mm_SilkScreen
- removed REF***: KiCad-Logo2_6mm_SilkScreen, Symbols:KiCad-Logo2_6mm_SilkScreen
- added C9: 4u7, Capacitors_THT:C_Rect_L7.0mm_W4.5mm_P5.00mm, F.Cu at (50.8, 95.9)
- added J3: Conn_02x22_Odd_Even, Pin_Headers:Pin_Header_Straight_2x22_Pitch2.00mm, F.Cu at (52.7, 144.4)
- moved TP1 8.52 mm to (62.2, 90.2)
Routing:
- net ~CS1~: track 56.5 -> 66.1 mm
- net ~CS3~: track 61.3 -> 70.9 mm, vias 2 -> 1
- net ~DASP~: track 29.8 -> 39.4 mm
- net BA0: track 46.1 -> 55.4 mm
- net BA1: track 52.2 -> 61.0 mm
- net ~RD~: track 62.6 -> 71.3 mm, vias 0 -> 2
- net ~BRESET~: track 101.0 -> 109.6 mm
- net INTRQ: track 50.1 -> 58.2 mm
- net BD7: track 34.1 -> 42.0 mm
- net /DMACK: track 7.67 -> 15.4 mm
- net BD6: track 34.1 -> 41.7 mm
- net BD5: track 34.1 -> 41.5 mm
- net BD8: track 20.7 -> 28.1 mm
- net BD0: track 33.9 -> 41.2 mm
- net BA2: track 63.1 -> 70.3 mm, vias 0 -> 1
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Other:
- board size 81.9 x 113 mm -> 83.8 x 113 mm
- board text added: "ATA/IDE Interface for Rosco_68k - v1.1 © Mark Murray 2021-03-25 https://certification.oshwa.org/uk000028.html"
- board text removed: "ATA/IDE Interface for Rosco_68k - v1.0 © Mark Murray 2021-03-20"

Commit message: PCB v1.1 RC1
Parts:
- added R5: 10k, Resistors_THT:R_Axial_DIN0207_L6.3mm_D2.5mm_P10.16mm_Horizontal, F.Cu at (94.0, 109.9)
- JP3, JP4: value SolderJumper_2_Open -> SolderJumper_2_Bridged; footprint Jumper:SolderJumper-2_P1.3mm_Open_Pad1.0x1.5mm -> Jumper:SolderJumper-2_P1.3mm_Bridged_Pad1.0x1.5mm
Connections:
- U1 pad 15: A8 -> (no net)
- U1 pad 18: (no net) -> A8
Routing:
- net A8: track 20.2 -> 27.9 mm
- net D0: track 27.1 -> 25.0 mm
- net ~SELECT~: track 19.5 -> 20.2 mm
- net D1: track 23.9 -> 24.6 mm
- net INTRQ: vias 2 -> 1

Commit message: Add some comments and correct dates.
Parts:
- C7: value 100u -> 10u
- C8: value 10u -> 100u
